File: Gilles/robot/Kicad_9.0/Kicad.kicad_sch (KiCad schematic)
At the start: 10 parts, among them J1 XH2.54_2P_socket, J2 XH2.54_2P_socket, J3 XH2.54_2P_socket, J4 Conn_01x04_Socket, SW1 SW_MINI_x1, U1 ESP32-C3_SUPERMINI, U2 L293D

Commit message: Add files via upload
Parts:
- added C1: C_Polarized, Gilles_Library:CP_8mm_3.5mm, symbol Device:C_Polarized
- added DH1, DH2, DH3, DH4: DRILL, Gilles_Library:DRILL_HOLE, symbol Gilles_Library:DRILL_HOLE
Connections:
- net GND: now also C1.2, DH1.1 (DH), DH2.1 (DH), DH3.1 (DH), DH4.1 (DH)
- net at J3.2, SW1.2 (B), SW1.3 (C): now also C1.1
