File: Gilles/telecommande/Kicad 9.0/telecommande.kicad_pcb (KiCad board)
At the start: 2 copper layers, 55 x 37 mm, 9 parts, among them J1 Conn_01x01_Pin, SW1 SW_MINI_x1, U1 ESP32-C3_SUPERMINI, U2 JOYSTICK 802

Commit message: Add files via upload
Parts:
- added DH1: DRILL, Gilles_Library:DRILL_HOLE, F.Cu at (75.5, 77.5)
- added DH2: DRILL, Gilles_Library:DRILL_HOLE, F.Cu at (125.5, 77.5)
- added DH3: DRILL, Gilles_Library:DRILL_HOLE, F.Cu at (75.5, 109.5)
- added DH4: DRILL, Gilles_Library:DRILL_HOLE, F.Cu at (125.5, 109.5)
- moved J1 6.08 mm to (119.7, 82.3)
- moved U1 2.11 mm to (86.7, 87.3)
- moved D3 0.70 mm to (104.0, 78.2)
Routing:
- net Net-(U1-GPIO2): track 22.8 -> 20.8 mm
- net Net-(U1-GPIO1): track 7.20 -> 5.43 mm
- net +3.3V: track 42.4 -> 40.6 mm
- net Net-(U1-GPIO0): track 20.9 -> 19.8 mm
- net Net-(D2-DIN): track 22.8 -> 21.8 mm
- net Net-(D1-DIN): track 28.4 -> 27.4 mm
- net +5V: track 41.3 -> 40.7 mm
- net Net-(SW1-A): track 4.80 -> 4.24 mm
