File: Gilles/telecommande/Kicad 9.0/telecommande.kicad_sch (KiCad schematic)
At the start: 9 parts, among them J1 Conn_01x01_Pin, SW1 SW_MINI_x1, U1 ESP32-C3_SUPERMINI, U2 JOYSTICK 802

Commit message: Add files via upload
Parts:
- added DH1, DH2, DH3, DH4: DRILL, Gilles_Library:DRILL_HOLE, symbol Gilles_Library:DRILL_HOLE
Connections:
- net GND: now also DH1.1 (DH), DH2.1 (DH), DH3.1 (DH), DH4.1 (DH)
